File: Schematics/Digit Display/digit display.kicad_sch (KiCad schematic)
At the start: 24 parts, among them J1 Conn_01x07

Commit message: Add files via upload
Parts:
- removed J1: Conn_01x07, pPSI:7 pin header, symbol Connector_Generic:Conn_01x07
- removed R17: 4.7k, pPSI:100ohm resistor, symbol pPSI:10kohm-Resistor
- added J1: 5-pin-header, pPSI:5 pin header, symbol pPSI:5-pin-header
Connections:
- net *OE is gone; now on net GND: ONES-SR1.13 (*OE), TENS-SR1.13 (*OE)
- net *SRCLR is gone; now on net VCC: ONES-SR1.10 (*SRCLR), TENS-SR1.10 (*SRCLR)
- net GND: now also J1.5 (Pin_5)
- net RCLK: now also J1.2 (Pin_2)
- net SER: now also J1.3 (Pin_3)
- net SRCLK: now also J1.1 (Pin_1)
- net VCC: now also J1.4 (Pin_4)
